File: cortex-debug/debugger-adapter.kicad_sch (KiCad schematic)
At the start: 4 parts

Commit message: Added part links
Parts:
- J2: Mates With (none) -> https://www.digikey.com/en/products/detail/cnc-tech/3230-10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
Changed lines of the file:
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@@
       (effects (font (size 1.27 1.27)) hide)
     )
-    (property "Datasheet" "" (at 175.26 78.74 0)
+    (property "Datasheet" "https://www.digikey.com/en/products/detail/cnc-tech/3240-10-00/3883786" (at 175.26 78.74 0)
+      (effects (font (size 1.27 1.27)) hide)
+    )
+    (property "Mates With" "https://www.digikey.com/en/products/detail/cnc-tech/3230-10-0102-00/3883464" (at 175.26 78.74 0)
       (effects (font (size 1.27 1.27)) hide)
     )
@@
       (effects (font (size 1.27 1.27)) hide)
     )
-    (property "Datasheet" "" (at 100.33 78.74 0)
+    (property "Datasheet" "https://www.digikey.com/en/products/detail/adam-tech/FCS-10-SG/9829300" (at 100.33 78.74 0)
       (effects (font (size 1.27 1.27)) hide)
     )
